File: Controller.brd (EAGLE design)
At the start: 100 x 66 mm, 20 parts, among them IC1 TB6612FNG

Commit message: initial board routing
Parts:
- moved R1_PAD_BACK 15.2 mm to (95.2, 63.5)
- moved R1_PAD_FRONT 15.2 mm to (95.2, 63.5)
- moved R2_PAD_BACK 15.2 mm to (80.0, 63.5)
- moved R2_PAD_FRONT 15.2 mm to (80.0, 63.5)
Routing:
- net VCC: track 0.00 -> 275.5 mm
- net GND: track 0.00 -> 182.8 mm, vias 0 -> 3
- net R_FWD: track 0.00 -> 124.6 mm, vias 0 -> 1
- net R_BCK: track 0.00 -> 82.0 mm, vias 0 -> 1
- net R_OUT1: track 0.00 -> 63.5 mm, vias 0 -> 1
- net L_OUT1: track 0.00 -> 61.9 mm, vias 0 -> 1
- net L_OUT2: track 0.00 -> 55.5 mm, vias 0 -> 1
- net R_OUT2: track 0.00 -> 51.3 mm, vias 0 -> 1
- net L_BCK: track 0.00 -> 47.7 mm, vias 0 -> 2
- net L_FWD: track 0.00 -> 37.9 mm
- net N$2: track 0.00 -> 17.8 mm
- net N$1: track 0.00 -> 17.8 mm
