File: Controller.brd (EAGLE design)
At the start: 100 x 66 mm, 21 parts, among them IC1 TB6612FNG

Commit message: fix button alignment
in other news, I got the 0.2 PCBs back today and they are **gorgeous**
Parts:
- moved L_BCK_BTN 1.27 mm to (12.7, 21.6)
- moved R2 1.27 mm to (22.9, 21.6)
Routing:
- net L_BCK: track 47.7 -> 46.4 mm
- net GND: track 182.8 -> 182.0 mm
Changed lines of the file:
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@@
 <attribute name="VALUE" x="18.95" y="66.3" size="0.0254" layer="27"/>
 </element>
-<element name="L_BCK_BTN" library="switch-omron" package="B3F-40XX" value="" x="12.7" y="20.32" smashed="yes">
-<attribute name="OC_NEWARK" value="36K3105" x="12.7" y="20.32" size="1.778" layer="27" display="off"/>
-<attribute name="MPN" value="B3F-4000" x="12.7" y="20.32" size="1.778" layer="27" display="off"/>
-<attribute name="MF" value="OMRON COMPONENTS USA" x="12.7" y="20.32" size="1.778" layer="27" display="off"/>
-<attribute name="OC_FARNELL" value="176434" x="12.7" y="20.32" size="1.778" layer="27" display="off"/>
-<attribute name="VALUE" x="9.525" y="15.24" size="1.27" layer="27" ratio="10"/>
+<element name="L_BCK_BTN" library="switch-omron" package="B3F-40XX" value="" x="12.7" y="21.59" smashed="yes">
+<attribute name="OC_NEWARK" value="36K3105" x="12.7" y="21.59" size="1.778" layer="27" display="off"/>
+<attribute name="MPN" value="B3F-4000" x="12.7" y="21.59" size="1.778" layer="27" display="off"/>
+<attribute name="MF" value="OMRON COMPONENTS USA" x="12.7" y="21.59" size="1.778" layer="27" display="off"/>
+<attribute name="OC_FARNELL" value="176434" x="12.7" y="21.59" size="1.778" layer="27" display="off"/>
+<attribute name="VALUE" x="9.525" y="16.51" size="1.27" layer="27" ratio="10"/>
 </element>
 <element name="L_FWD_BTN" library="switch-omron" package="B3F-40XX" value="" x="12.7" y="45.72" smashed="yes">
@@
 <attribute name="VALUE" x="92.61" y="66.3" size="0.0254" layer="27"/>
 </element>
-<element name="R2" library="rcl" package="R0805" value="10k" x="22.86" y="20.32" smashed="yes" rot="MR0"/>
+<element name="R2" library="rcl" package="R0805" value="10k" x="22.86" y="21.59" smashed="yes" rot="MR0"/>
 <element name="R2_PAD_BACK" library="wirepad" package="5-2,5" value="WIREPADSMD5-2,5" x="82.55" y="63.5" smashed="yes" rot="MR0">
 <attribute name="VALUE" x="82.65" y="66.3" size="0.0254" layer="28" rot="MR0"/>
@@
 <wire x1="10.16" y1="43.2308" x2="6.4516" y2="43.2308" width="0.4064" layer="16"/>
 <wire x1="33.02" y1="7.874" x2="28.9052" y2="7.874" width="0.4064" layer="16"/>
-<wire x1="28.9052" y1="7.874" x2="18.9484" y2="17.8308" width="0.4064" layer="16"/>
-<wire x1="18.9484" y1="17.8308" x2="10.2108" y2="17.8308" width="0.4064" layer="16"/>
-<wire x1="10.2108" y1="17.8308" x2="6.4516" y2="17.8308" width="0.4064" layer="16"/>
+<wire x1="28.9052" y1="7.874" x2="18.9484" y2="19.1008" width="0.4064" layer="16"/>
+<wire x1="18.9484" y1="19.1008" x2="10.2108" y2="19.1008" width="0.4064" layer="16"/>
+<wire x1="10.2108" y1="19.1008" x2="6.4516" y2="19.1008" width="0.4064" layer="16"/>
 <wire x1="18.9484" y1="43.2308" x2="12.7508" y2="43.2308" width="0.4064" layer="16"/>
 <wire x1="12.7508" y1="43.2308" x2="12.7" y2="43.18" width="0.4064" layer="16"/>
-<wire x1="10.2108" y1="17.8308" x2="10.16" y2="17.78" width="0.4064" layer="16"/>
-<wire x1="10.16" y1="17.78" x2="10.16" y2="43.2308" width="0.4064" layer="16"/>
+<wire x1="10.2108" y1="19.1008" x2="10.16" y2="19.05" width="0.4064" layer="16"/>
+<wire x1="10.16" y1="19.05" x2="10.16" y2="43.2308" width="0.4064" layer="16"/>
 <wire x1="81.3816" y1="43.2308" x2="93.8784" y2="43.2308" width="0.4064" layer="16"/>
 <wire x1="81.3816" y1="19.1008" x2="93.8784" y2="19.1008" width="0.4064" layer="16"/>
@@
 <wire x1="54.4197125" y1="31.4002875" x2="54.425" y2="31.395" width="0.4064" layer="16"/>
 <wire x1="54.425" y1="31.395" x2="54.425" y2="30.745" width="0.4064" layer="16"/>
-<wire x1="23.81" y1="20.32" x2="36.035" y2="32.545" width="0.4064" layer="16"/>
+<wire x1="23.81" y1="21.59" x2="36.035" y2="32.545" width="0.4064" layer="16"/>
 <wire x1="36.035" y1="32.545" x2="36.185" y2="32.695" width="0.4064" layer="16"/>
 <wire x1="36.185" y1="32.695" x2="47.175" y2="32.695" width="0.4064" layer="16"/>
@@
 <contactref element="R2" pad="2"/>
 <contactref element="IC1" pad="22"/>
-<wire x1="21.91" y1="20.32" x2="21.4376" y2="20.32" width="0.8128" layer="16"/>
-<wire x1="21.4376" y1="20.32" x2="18.9484" y2="22.8092" width="0.8128" layer="16"/>
-<wire x1="21.91" y1="20.32" x2="21.91" y2="26.35" width="0.4064" layer="16"/>
+<wire x1="21.91" y1="21.59" x2="21.4376" y2="21.59" width="0.8128" layer="16"/>
+<wire x1="21.4376" y1="21.59" x2="18.9484" y2="24.0792" width="0.8128" layer="16"/>
+<wire x1="21.91" y1="21.59" x2="21.91" y2="26.35" width="0.4064" layer="16"/>
 <wire x1="21.91" y1="26.35" x2="20.32" y2="27.94" width="0.4064" layer="16"/>
 <via x="20.32" y="27.94" extent="1-16" drill="0.6" shape="square"/>
